Commit message: add mimic tag for palm joint

File: robotiq_3f_gripper_visualization/cfg/robotiq-3f-gripper_articulated_macro.xacro (robot description, xacro)
@@ -51,4 +51,5 @@
 			<origin xyz="-0.0455 0.0214 -0.036" rpy="0 3.1416 -1.57"/>
 			<limit lower="-0.192" upper="0.1784" effort="100" velocity="100"/>
+			<mimic joint="${prefix}palm_finger_1_joint" multiplier="-1"/>
 		</joint>
 		<joint name="${prefix}palm_finger_middle_joint" type="fixed">
